File: design_files/ASL1201.sch (EAGLE design)
At the start: 2 parts, among them J1 LPPB051NGCN-RC, J2 S2B-PH-SM4

Commit message: update format
Parts:
- added J3, J4: PIN_1X.1"1, tinycircuits:PIN_1X.1"1
- J2: value S2B-PH-SM4 -> SM02B-SRSS-TB(LF)(SN); device tinycircuits:AS-ITM-00043 -> tinycircuits:AS-ITM-00231
Connections:
- removed net GND: J1.2, J2.1
- removed net VCC: J1.1, J2.2
- new net N$1: J1.1, J2.1, J4.1
- new net N$2: J1.2, J2.2, J3.1
Other:
- note added: "2"
- note removed: "1"
- moved on the sheet: J2
Changed lines of the file:
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@@
 <?xml version="1.0" encoding="utf-8"?>
 <!DOCTYPE eagle SYSTEM "eagle.dtd">
-<eagle version="6.2">
+<eagle version="6.3">
 <drawing>
 <settings>
@@
 <layer number="106" name="bPlate" color="7" fill="1" visible="yes" active="yes"/>
 <layer number="107" name="Crop" color="7" fill="1" visible="yes" active="yes"/>
+<layer number="108" name="fp8" color="7" fill="1" visible="yes" active="yes"/>
+<layer number="109" name="fp9" color="7" fill="1" visible="yes" active="yes"/>
+<layer number="110" name="fp0" color="7" fill="1" visible="yes" active="yes"/>
+<layer number="111" name="LPC17xx" color="7" fill="1" visible="yes" active="yes"/>
+<layer number="112" name="tSilk" color="7" fill="1" visible="yes" active="yes"/>
 <layer number="116" name="Patch_BOT" color="7" fill="1" visible="yes" active="yes"/>
 <layer number="121" name="_tsilk" color="7" fill="1" visible="yes" active="yes"/>
 <layer number="122" name="_bsilk" color="7" fill="1" visible="yes" active="yes"/>
+<layer number="123" name="tTestmark" color="7" fill="1" visible="yes" active="yes"/>
+<layer number="124" name="bTestmark" color="7" fill="1" visible="yes" active="yes"/>
+<layer number="125" name="_tNames" color="7" fill="1" visible="yes" active="yes"/>
+<layer number="126" name="_bNames" color="7" fill="1" visible="yes" active="yes"/>
+<layer number="127" name="_tValues" color="7" fill="1" visible="yes" active="yes"/>
+<layer number="128" name="_bValues" color="7" fill="1" visible="yes" active="yes"/>
+<layer number="131" name="tAdjust" color="7" fill="1" visible="yes" active="yes"/>
+<layer number="132" name="bAdjust" color="7" fill="1" visible="yes" active="yes"/>
 <layer number="144" name="Drill_legend" color="7" fill="1" visible="yes" active="yes"/>
 <layer number="151" name="HeatSink" color="7" fill="1" visible="yes" active="yes"/>
+<layer number="152" name="_bDocu" color="7" fill="1" visible="yes" active="yes"/>
+<layer number="199" name="Contour" color="7" fill="1" visible="yes" active="yes"/>
 <layer number="200" name="200bmp" color="7" fill="1" visible="yes" active="yes"/>
 <layer number="201" name="201bmp" color="7" fill="1" visible="yes" active="yes"/>
@@
 <layer number="223" name="223bmp" color="7" fill="1" visible="yes" active="yes"/>
 <layer number="224" name="224bmp" color="7" fill="1" visible="yes" active="yes"/>
+<layer number="248" name="Housing" color="7" fill="1" visible="yes" active="yes"/>
+<layer number="249" name="Edge" color="7" fill="1" visible="yes" active="yes"/>
 <layer number="250" name="Descript" color="7" fill="1" visible="yes" active="yes"/>
 <layer number="251" name="SMDround" color="7" fill="1" visible="yes" active="yes"/>
@@
 <part name="FRAME1" library="tinycircuits" deviceset="FRAME_TINYCIRCUITS_B_L" device=""/>
 <part name="J1" library="tinycircuits" deviceset="AS-ITM-00037" device="" value="LPPB051NGCN-RC"/>
-<part name="J2" library="tinycircuits" deviceset="AS-ITM-00043" device="" value="S2B-PH-SM4"/>
+<part name="J2" library="tinycircuits" deviceset="AS-ITM-00231" device="" value="SM02B-SRSS-TB(LF)(SN)"/>
+<part name="J4" library="tinycircuits" deviceset="PIN_1X.1&quot;" device="1"/>
+<part name="J3" library="tinycircuits" deviceset="PIN_1X.1&quot;" device="1"/>
 </parts>
 <sheets>
@@
 <text x="340.868" y="17.272" size="3.556" layer="94" font="vector">TinyLily Power Adapter Bd</text>
 <text x="327.152" y="6.35" size="3.556" layer="94" font="vector">AS-SCH-ASL1201</text>
-<text x="416.56" y="6.858" size="3.556" layer="94" font="vector">1</text>
+<text x="416.56" y="6.858" size="3.556" layer="94" font="vector">2</text>
 <text x="45.72" y="35.56" size="3.048" layer="91">Released under the Creative Commons Attribution Share-Alike 3.0 License</text>
 <text x="45.72" y="30.48" size="3.048" layer="91">http://creativecommons.org/licenses/by-sa/3.0</text>
@@
 <attribute name="VALUE" x="231.14" y="132.08" size="1.778" layer="96"/>
 </instance>
-<instance part="J2" gate="G$1" x="205.74" y="147.32" smashed="yes" rot="R180">
-<attribute name="NAME" x="209.042" y="151.892" size="1.778" layer="95" rot="R180"/>
-<attribute name="VALUE" x="216.154" y="141.732" size="1.778" layer="96" rot="R180"/>
-</instance>
+<instance part="J2" gate="G$1" x="205.74" y="144.78" rot="MR0"/>
+<instance part="J4" gate="G$1" x="218.44" y="149.86" rot="R270"/>
+<instance part="J3" gate="G$1" x="218.44" y="142.24" rot="R90"/>
 </instances>
 <busses>
 </busses>
 <nets>
-<net name="VCC" class="0">
+<net name="N$1" class="0">
 <segment>
-<wire x1="233.68" y1="147.32" x2="215.9" y2="147.32" width="0.1524" layer="91"/>
-<label x="222.504" y="147.574" size="1.778" layer="95"/>
+<pinref part="J2" gate="G$1" pin="1"/>
+<pinref part="J4" gate="G$1" pin="1"/>
+<wire x1="215.9" y1="147.32" x2="218.44" y2="147.32" width="0.1524" layer="91"/>
+<wire x1="218.44" y1="147.32" x2="218.44" y2="149.86" width="0.1524" layer="91"/>
 <pinref part="J1" gate="G$1" pin="1"/>
-<pinref part="J2" gate="G$1" pin="2"/>
+<wire x1="218.44" y1="147.32" x2="233.68" y2="147.32" width="0.1524" layer="91"/>
+<junction x="218.44" y="147.32"/>
 </segment>
 </net>
-<net name="GND" class="0">
+<net name="N$2" class="0">
 <segment>
 <pinref part="J1" gate="G$1" pin="2"/>
-<pinref part="J2" gate="G$1" pin="1"/>
-<wire x1="215.9" y1="144.78" x2="233.68" y2="144.78" width="0.1524" layer="91"/>
-<label x="222.504" y="145.034" size="1.778" layer="95"/>
+<pinref part="J2" gate="G$1" pin="2"/>
+<wire x1="233.68" y1="144.78" x2="218.44" y2="144.78" width="0.1524" layer="91"/>
+<pinref part="J3" gate="G$1" pin="1"/>
+<wire x1="218.44" y1="144.78" x2="215.9" y2="144.78" width="0.1524" layer="91"/>
+<wire x1="218.44" y1="144.78" x2="218.44" y2="142.24" width="0.1524" layer="91"/>
+<junction x="218.44" y="144.78"/>
 </segment>
 </net>
